File: kicad/Ordered/V1/BMS.sch (KiCad schematic (older format))
At the start: 8 parts, among them J4 Conn_01x02_Female, SW1 SW_SPDT, U7 LM3671

Commit message: code updates
Parts:
- C19: value 4.7uF -> 0.1uF
- C21: value 10uF -> C
- L4: value 2.2uH -> INDUCTOR
Changed lines of the file:
@@
 P 4400 2050
 F 0 "C19" H 4492 2096 50  0000 L CNN
-F 1 "4.7uF" H 4492 2005 50  0000 L CNN
+F 1 "0.1uF" H 4492 2005 50  0000 L CNN
 F 2 "Capacitor_SMD:C_0805_2012Metric" H 4400 2050 50  0001 C CNN
 F 3 "~" H 4400 2050 50  0001 C CNN
@@
 P 6050 1850
 F 0 "L4" H 6050 2065 50  0000 C CNN
-F 1 "2.2uH" H 6050 1974 50  0000 C CNN
+F 1 "INDUCTOR" H 6050 1974 50  0000 C CNN
 F 2 "Inductor_SMD:L_0805_2012Metric" H 6050 1850 50  0001 C CNN
 F 3 "~" H 6050 1850 50  0001 C CNN
@@
 P 6600 2000
 F 0 "C21" H 6715 2046 50  0000 L CNN
-F 1 "10uF" H 6715 1955 50  0000 L CNN
+F 1 "C" H 6715 1955 50  0000 L CNN
 F 2 "Capacitor_SMD:C_0805_2012Metric" H 6638 1850 50  0001 C CNN
 F 3 "~" H 6600 2000 50  0001 C CNN
