File: kicad/Ordered/V1/bullercounter - Copy.sch (KiCad schematic (older format))
At the start: 49 parts, among them J1 USB_B_Micro, J2 Conn_ARM_JTAG_SWD_10, J3 Serial, J5 TP, SW3 Switch, SW4 Switch, SW5 Switch, U1 MCP6421, U2 ATSAMD21G18A-AUT, U3 LSM6DS3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

Commit message: code updates
Parts:
- removed C10, C6, C7: 100pF, Capacitor_SMD:C_0805_2012Metric, symbol Device:C_Small
- removed H1, H2, H3, H4: MountingHole, MountingHole:MountingHole_2.7mm, symbol Mechanical:MountingHole
- removed R13, R14, R15: 10k, Resistor_SMD:R_0603_1608Metric, symbol Device:R
- removed U5: MO043803_4.5mm, CustomFP:MO043803_4.5mm, symbol CustomComponents:MO043803_4.5mm
- added C6: 82n, Capacitor_SMD:C_0805_2012Metric, symbol Device:C
- added MK1: Mic, Connector_PinHeader_2.54mm:PinHeader_1x02_P2.54mm_Vertical, symbol Device:Microphone_Condenser
- added SW2: Switch, EbayParts:Tact_SMD_Switch, symbol weatherStation-cache:Switch_SW_Push
- J3: footprint CustomFP:SMD_1Pin_1.5mm -> Connector_PinHeader_2.54mm:PinHeader_1x02_P2.54mm_Vertical
- J5: footprint CustomFP:SMD_1Pin_1.5mm -> Connector_PinHeader_1.27mm:PinHeader_1x02_P1.27mm_Vertical
Connections:
- net labels removed: BattADC, BattPwr, IMU_INT2
- wire segments 106 -> 95
- no-connect marks 4 -> 5
Other:
- note removed: "Anode +\n\nCathoode -"
